File: droninho.kicad_sch (KiCad schematic)
At the start: 34 parts, among them J6 I2C, J7 TXD0/RXD0, J8 I2C, Q1 Si2300DS, Q2 Si2300DS, Q3 Si2300DS, Q4 Si2300DS, SW1 KMR241G LFS, U1 AMS1117-3.3, U2 MPU9250/6500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

Commit message: add manufacturer and part number for BOM.
Parts:
- added H1: MountingHole_Pad_MP, MountingHole:MountingHole_2.2mm_M2_DIN965_Pad, symbol Mechanical:MountingHole_Pad_MP
- C1: Designator (none) -> C1; Manufacturer (none) -> Murata Electronics; Mfg Part # (none) -> GRM21BR61A226ME51L; Package/Footprint (none) -> 0805; Type (none) -> SMD
- C2: Designator (none) -> C2; Manufacturer (none) -> Murata Electronics; Mfg Part # (none) -> GRM21BR61A226ME51L; Package/Footprint (none) -> 0805; Type (none) -> SMD
- C3: value 0.1uF/50V(10%) -> 0.1uF/10V(5%); Designator (none) -> C3; Manufacturer (none) -> Murata Electronics; Mfg Part # (none) -> GRM21B7U1A104JA01L; Package/Footprint (none) -> 0805; Type (none) -> SMD
- D1: Designator (none) -> D1; Manufacturer (none) -> Wurth Elektronik; Mfg Part # (none) -> 150080RS75000; Package/Footprint (none) -> 0805; Type (none) -> SMD
- D2: Designator (none) -> D2; Manufacturer (none) -> Broadcom / Avago; Mfg Part # (none) -> HSMW-C170; Package/Footprint (none) -> 0805; Type (none) -> SMD
- D3: Designator (none) -> D3; Manufacturer (none) -> Broadcom / Avago; Mfg Part # (none) -> HSMW-C170; Package/Footprint (none) -> 0805; Type (none) -> SMD
- D4: Designator (none) -> D4; Manufacturer (none) -> Broadcom / Avago; Mfg Part # (none) -> HSMW-C170; Package/Footprint (none) -> 0805; Type (none) -> SMD
- D5: Designator (none) -> D5; Manufacturer (none) -> Broadcom / Avago; Mfg Part # (none) -> HSMW-C170; Package/Footprint (none) -> 0805; Type (none) -> SMD
- D6: Designator (none) -> D6; Manufacturer (none) -> Diotec Semiconductor; Mfg Part # (none) -> 1N4148W; Package/Footprint (none) -> SOD-123F; Type (none) -> SMD
- D7: Designator (none) -> D7; Manufacturer (none) -> Diotec Semiconductor; Mfg Part # (none) -> 1N4148W; Package/Footprint (none) -> SOD-123F; Type (none) -> SMD
- D8: Designator (none) -> D8; Manufacturer (none) -> Diotec Semiconductor; Mfg Part # (none) -> 1N4148W; Package/Footprint (none) -> SOD-123F; Type (none) -> SMD
- D9: Designator (none) -> D9; Manufacturer (none) -> Diotec Semiconductor; Mfg Part # (none) -> 1N4148W; Package/Footprint (none) -> SOD-123F; Type (none) -> SMD
- Q1: Designator (none) -> Q1; Manufacturer (none) -> Vishay; Mfg Part # (none) -> SI2300DS-T1-BE3; Package/Footprint (none) -> SOT-23 (TO-236); Type (none) -> SMD
- Q2: Designator (none) -> Q2; Manufacturer (none) -> Vishay; Mfg Part # (none) -> SI2300DS-T1-BE3; Package/Footprint (none) -> SOT-23 (TO-236); Type (none) -> SMD
- Q3: Designator (none) -> Q3; Manufacturer (none) -> Vishay; Mfg Part # (none) -> SI2300DS-T1-BE3; Package/Footprint (none) -> SOT-23 (TO-236); Type (none) -> SMD
- Q4: Designator (none) -> Q4; Manufacturer (none) -> Vishay; Mfg Part # (none) -> SI2300DS-T1-BE3; Package/Footprint (none) -> SOT-23 (TO-236); Type (none) -> SMD
- R1: value 10K(5%) -> 10K(1%); Designator (none) -> R1; Manufacturer (none) -> Panasonic; Mfg Part # (none) -> ERJ-6ENF1002V; Package/Footprint (none) -> 0805; Type (none) -> SMD
- R2: value 10K(5%) -> 10K(1%); Designator (none) -> R2; Manufacturer (none) -> Panasonic; Mfg Part # (none) -> ERJ-6ENF1002V; Package/Footprint (none) -> 0805; Type (none) -> SMD
- R3: value 10K(5%) -> 10K(1%); Designator (none) -> R3; Manufacturer (none) -> Panasonic; Mfg Part # (none) -> ERJ-6ENF1002V; Package/Footprint (none) -> 0805; Type (none) -> SMD
- R4: value 10K(5%) -> 10K(1%); Designator (none) -> R4; Manufacturer (none) -> Panasonic; Mfg Part # (none) -> ERJ-6ENF1002V; Package/Footprint (none) -> 0805; Type (none) -> SMD
- R5: value 10K(5%) -> 10K(1%); Designator (none) -> R5; Manufacturer (none) -> Panasonic; Mfg Part # (none) -> ERJ-6ENF1002V; Package/Footprint (none) -> 0805; Type (none) -> SMD

Commit message: BOM updated.
Parts:
- removed H1: MountingHole_Pad_MP, MountingHole:MountingHole_2.2mm_M2_DIN965_Pad, symbol Mechanical:MountingHole_Pad_MP
- J6: Designator (none) -> J6; Manufacturer (none) -> Molex; Mfg Part # (none) -> 502603-0470; Package/Footprint (none) -> 4POS; Type (none) -> THT
- J7: Designator (none) -> J7; Manufacturer (none) -> Molex; Mfg Part # (none) -> 502603-0470; Package/Footprint (none) -> 4POS; Type (none) -> THT
- J8: Designator (none) -> J8; Manufacturer (none) -> Molex; Mfg Part # (none) -> 502603-0470; Package/Footprint (none) -> 4POS; Type (none) -> THT
- SW1: Designator (none) -> SW1; Manufacturer (none) -> C&K; Mfg Part # (none) -> KMR241G LFS; Package/Footprint (none) -> SW_Push_1P1T_NO_CK_KMR2; Type (none) -> SMT
Changed lines of the file:
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@@
 			)
 		)
+		(property "Manufacturer" "Molex"
+			(at 250.19 66.04 0)
+			(effects
+				(font
+					(size 1.27 1.27)
+				)
+				(hide yes)
+			)
+		)
+		(property "Mfg Part #" "502603-0470"
+			(at 250.19 66.04 0)
+			(effects
+				(font
+					(size 1.27 1.27)
+				)
+				(hide yes)
+			)
+		)
+		(property "Package/Footprint" "4POS"
+			(at 250.19 66.04 0)
+			(effects
+				(font
+					(size 1.27 1.27)
+				)
+				(hide yes)
+			)
+		)
+		(property "Type" "THT"
+			(at 250.19 66.04 0)
+			(effects
+				(font
+					(size 1.27 1.27)
+				)
+				(hide yes)
+			)
+		)
+		(property "Designator" "J7"
+			(at 250.19 66.04 0)
+			(effects
+				(font
+					(size 1.27 1.27)
+				)
+				(hide yes)
+			)
+		)
 		(pin "1"
 		)
@@
 	)
 	(symbol
-		(lib_id "Mechanical:MountingHole_Pad_MP")
-		(at 107.95 22.86 0)
-		(unit 1)
-		(exclude_from_sim no)
-		(in_bom no)
-		(on_board yes)
-		(dnp no)
-		(fields_autoplaced yes)
-		(property "Reference" "H1"
-			(at 110.49 20.3199 0)
-			(effects
-				(font
-					(size 1.27 1.27)
-				)
-				(justify left)
-			)
-		)
-		(property "Value" "MountingHole_Pad_MP"
-			(at 110.49 22.8599 0)
-			(effects
-				(font
-					(size 1.27 1.27)
-				)
-				(justify left)
-			)
-		)
-		(property "Footprint" "MountingHole:MountingHole_2.2mm_M2_DIN965_Pad"
-			(at 107.95 22.86 0)
-			(effects
-				(font
-					(size 1.27 1.27)
-				)
-				(hide yes)
-			)
-		)
-		(property "Datasheet" "~"
-			(at 107.95 22.86 0)
-			(effects
-				(font
-					(size 1.27 1.27)
-				)
-				(hide yes)
-			)
-		)
-		(property "Description" "Mounting Hole with connection as pad named MP"
-			(at 107.95 22.86 0)
-			(effects
-				(font
-					(size 1.27 1.27)
-				)
-				(hide yes)
-			)
-		)
-		(property "Manufacturer" ""
-			(at 107.95 22.86 0)
-			(effects
-				(font
-					(size 1.27 1.27)
-				)
-				(hide yes)
-			)
-		)
-		(property "Mfg Part #" ""
-			(at 107.95 22.86 0)
-			(effects
-				(font
-					(size 1.27 1.27)
-				)
-				(hide yes)
-			)
-		)
-		(property "Package/Footprint" ""
-			(at 107.95 22.86 0)
-			(effects
-				(font
-					(size 1.27 1.27)
-				)
-				(hide yes)
-			)
-		)
-		(property "Type" ""
-			(at 107.95 22.86 0)
-			(effects
-				(font
-					(size 1.27 1.27)
-				)
-				(hide yes)
-			)
-		)
-		(property "Designator" ""
-			(at 107.95 22.86 0)
-			(effects
-				(font
-					(size 1.27 1.27)
-				)
-				(hide yes)
-			)
-		)
-		(pin "MP"
-		)
-		(instances
-			(project ""
-				(path "/50215636-8ce2-4b01-ade7-3715bffabe9d"
-					(reference "H1")
-					(unit 1)
-				)
-			)
-		)
-	)
-	(symbol
 		(lib_id "Device:R_US")
 		(at 29.21 39.37 0)
@@
 			)
 		)
+		(property "Manufacturer" "Molex"
+			(at 251.46 30.48 0)
+			(effects
+				(font
+					(size 1.27 1.27)
+				)
+				(hide yes)
+			)
+		)
+		(property "Mfg Part #" "502603-0470"
+			(at 251.46 30.48 0)
+			(effects
+				(font
+					(size 1.27 1.27)
+				)
+				(hide yes)
+			)
+		)
+		(property "Package/Footprint" "4POS"
+			(at 251.46 30.48 0)
+			(effects
+				(font
+					(size 1.27 1.27)
+				)
+				(hide yes)
+			)
+		)
+		(property "Type" "THT"
+			(at 251.46 30.48 0)
+			(effects
+				(font
+					(size 1.27 1.27)
+				)
+				(hide yes)
+			)
+		)
+		(property "Designator" "J6"
+			(at 251.46 30.48 0)
+			(effects
+				(font
+					(size 1.27 1.27)
+				)
+				(hide yes)
+			)
+		)
 		(pin "1"
 		)
@@
 			)
 		)
+		(property "Manufacturer" "Molex"
+			(at 250.19 102.87 0)
+			(effects
+				(font
+					(size 1.27 1.27)
+				)
+				(hide yes)
+			)
+		)
+		(property "Mfg Part #" "502603-0470"
+			(at 250.19 102.87 0)
+			(effects
+				(font
+					(size 1.27 1.27)
+				)
+				(hide yes)
+			)
+		)
+		(property "Package/Footprint" "4POS"
+			(at 250.19 102.87 0)
+			(effects
+				(font
+					(size 1.27 1.27)
+				)
+				(hide yes)
+			)
+		)
+		(property "Type" "THT"
+			(at 250.19 102.87 0)
+			(effects
+				(font
+					(size 1.27 1.27)
+				)
+				(hide yes)
+			)
+		)
+		(property "Designator" "J8"
+			(at 250.19 102.87 0)
+			(effects
+				(font
+					(size 1.27 1.27)
+				)
+				(hide yes)
+			)
+		)
 		(pin "1"
 		)
@@
 			(at 256.54 130.81 0)
 			(effects
+				(font
+					(size 1.27 1.27)
+				)
+				(hide yes)
+			)
+		)
+		(property "Manufacturer" "C&K"
+			(at 256.54 130.81 0)
+			(effects
+				(font
+					(size 1.27 1.27)
+				)
+				(hide yes)
+			)
+		)
+		(property "Mfg Part #" "KMR241G LFS"
+			(at 256.54 130.81 0)
+			(effects
+				(font
+					(size 1.27 1.27)
+				)
+				(hide yes)
+			)
+		)
+		(property "Package/Footprint" "SW_Push_1P1T_NO_CK_KMR2"
+			(at 256.54 130.81 0)
+			(effects
+				(font
+					(size 1.27 1.27)
+				)
+				(hide yes)
+			)
+		)
+		(property "Type" "SMT"
+			(at 256.54 130.81 0)
+			(effects
+				(font
+					(size 1.27 1.27)
+				)
+				(hide yes)
+			)
+		)
+		(property "Designator" "SW1"
+			(at 256.54 130.81 0)
+			(effects

Commit message: first commit
Parts:
- removed U2: MPU9250/6500, Library:MPU-9250-6500, symbol Library:MPU-9250-6500
- added C4, C5, C6, C7: 0.1uF/10V(5%), Capacitor_SMD:C_0402_1005Metric, symbol Device:C_Small
- added C8: C_Small_US, Capacitor_SMD:C_0201_0603Metric, symbol Device:C_Small_US
- added U2: TLV70218_SOT23-5, Package_TO_SOT_SMD:SOT-23-5, symbol Regulator_Linear:TLV70218_SOT23-5
- added U8: ICM-20948, Sensor_Motion:InvenSense_QFN-24_3x3mm_P0.4mm, symbol Sensor_Motion:ICM-20948
Connections:
- net GND: now also C4.1, C5.1, C6.1, C7.1, C8.2, U2.2 (GND), U8.18 (GND), U8.20 (GND)
- net SCL: now also U8.23 (SCL/SCLK)
- net SDA: now also U8.24 (SDA/SDI)
- new net: C7.2, U2.1 (IN), U2.3 (EN)
- new net: C4.2, U8.10 (REGOUT)
- new net: C6.2, U8.13 (VDD)
- new net: C5.2, U8.8 (VDDIO)
- new net: C8.1, U2.5 (OUT)
Other:
- note added: "Voltage Regulator 1.8v"
- note added: "Voltage Regulator 3.3v"
- note removed: "Power Regulator"
- moved on the sheet: C1, C2, D1, D2, D3, D4, D5, H3, H4, R1, R2, R3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

Commit message: first commit
Parts:
- removed C3: 0.1uF/10V(5%), Capacitor_SMD:C_0805_2012Metric_Pad1.18x1.45mm_HandSolder, symbol Device:C_Small
- removed C4, C5, C6, C7: 0.1uF/10V(5%), Capacitor_SMD:C_0402_1005Metric, symbol Device:C_Small
- removed C8: C_Small_US, Capacitor_SMD:C_0201_0603Metric, symbol Device:C_Small_US
- removed J6, J8: I2C, Connector_PinHeader_2.54mm:PinHeader_1x04_P2.54mm_Vertical, symbol Connector:Conn_01x04_Pin
- removed J7: TXD0/RXD0, Connector_PinHeader_2.54mm:PinHeader_1x04_P2.54mm_Vertical, symbol Connector:Conn_01x04_Pin
- removed SW1: KMR241G LFS, Button_Switch_SMD:SW_Push_1P1T_NO_CK_KMR2, symbol Switch:SW_Push
- removed U2: TLV70218_SOT23-5, Package_TO_SOT_SMD:SOT-23-5, symbol Regulator_Linear:TLV70218_SOT23-5
- removed U3: ESP32 ESP-WROOM-32 DEVKit V1, Library:ESP32_30pin vertical WIFI, symbol Library:ESP32_30Pin_vertical_WIFI
- removed U8: ICM-20948, Sensor_Motion:InvenSense_QFN-24_3x3mm_P0.4mm, symbol Sensor_Motion:ICM-20948
- added J1: Conn_01x06_Socket, Connector_PinSocket_1.00mm:PinSocket_1x06_P1.00mm_Vertical, symbol Connector:Conn_01x06_Socket
Connections:
- net GND: now also J1.2 (Pin_2)
- net PWM1: now also J1.3 (Pin_3)
- net PWM2: now also J1.4 (Pin_4)
- net PWM3: now also J1.5 (Pin_5)
- net PWM4: now also J1.6 (Pin_6)
- no-connect marks 22 -> 0
Other:
- note removed: "Conector I2C"
- note removed: "Conector TXD0/RXD0"
- note removed: "Conector TXD2/RXD2"
- note removed: "Processamento e controle"
- note removed: "Push Button"
- note removed: "Sensores"
- note removed: "Voltage Regulator 1.8v"

Commit message: driver PCB ready
Parts:
- removed U4, U5, U6, U7: Through Hole Connector, Library:Connector_Motor, symbol Library:Connector_Motor
- added J2, J3, J4, J5: Conn_01x02_Socket, Connector_Hirose:Hirose_DF13-02P-1.25DSA_1x02_P1.25mm_Vertical, symbol Connector:Conn_01x02_Socket
- J1: footprint Connector_PinSocket_1.00mm:PinSocket_1x06_P1.00mm_Vertical -> Connector_Hirose:Hirose_DF13-06P-1.25DSA_1x06_P1.25mm_Vertical
Connections:
- net +3.3V: now also J1.1 (Pin_1), J2.2 (Pin_2), J3.2 (Pin_2), J4.2 (Pin_2), J5.2 (Pin_2)
- net M1-: now also J2.1 (Pin_1)
- net M2-: now also J3.1 (Pin_1)
- net M3-: now also J4.1 (Pin_1)
- net M4-: now also J5.1 (Pin_1)
Other:
- moved on the sheet: D2, D3, D4, D5, H3, H4, J1, R2, R3, R4, R5

Commit message: small updates
Other:
- moved on the sheet: C1, C2, D1, D2, D3, D4, D5, D6, D7, D8, D9, H3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

Commit message: driver finalizado.
Parts:
- J1: footprint Connector_Hirose:Hirose_DF13-06P-1.25DSA_1x06_P1.25mm_Vertical -> Connector_JST:JST_PH_B6B-PH-K_1x06_P2.00mm_Vertical; Designator (none) -> J1; Manufacturer (none) -> JST Commercial; Mfg Part # (none) -> BM06B-PASS-TF(LF)(SN); Package/Footprint (none) -> 6POS; Type (none) -> thru-hole
- J2: footprint Connector_Hirose:Hirose_DF13-02P-1.25DSA_1x02_P1.25mm_Vertical -> Connector_JST:JST_PH_B2B-PH-K_1x02_P2.00mm_Vertical; Designator (none) -> J2; Manufacturer (none) -> JST Commercial; Mfg Part # (none) -> BM02B-PASS-TF(LF)(SN); Package/Footprint (none) -> 2POS; Type (none) -> thru-hole
- J3: footprint Connector_Hirose:Hirose_DF13-02P-1.25DSA_1x02_P1.25mm_Vertical -> Connector_JST:JST_PH_B2B-PH-K_1x02_P2.00mm_Vertical; Designator (none) -> J3; Manufacturer (none) -> JST Commercial; Mfg Part # (none) -> BM02B-PASS-TF(LF)(SN); Package/Footprint (none) -> 2POS; Type (none) -> thru-hole
- J4: footprint Connector_Hirose:Hirose_DF13-02P-1.25DSA_1x02_P1.25mm_Vertical -> Connector_JST:JST_PH_B2B-PH-K_1x02_P2.00mm_Vertical; Designator (none) -> J4; Manufacturer (none) -> JST Commercial; Mfg Part # (none) -> BM02B-PASS-TF(LF)(SN); Package/Footprint (none) -> 2POS; Type (none) -> thru-hole
- J5: footprint Connector_Hirose:Hirose_DF13-02P-1.25DSA_1x02_P1.25mm_Vertical -> Connector_JST:JST_PH_B2B-PH-K_1x02_P2.00mm_Vertical; Designator (none) -> J5; Manufacturer (none) -> JST Commercial; Mfg Part # (none) -> BM02B-PASS-TF(LF)(SN); Package/Footprint (none) -> 2POS; Type (none) -> thru-hole
- U1: Designator (none) -> U1; Manufacturer (none) -> Texas Instruments; Mfg Part # (none) -> LM1117MPX-3.3/NOPB; Package/Footprint (none) -> SOT-223-4; Type (none) -> SMD
